Commit message: moveit

File: so_arm_100_description/urdf/so_arm_100_5dof_arm.urdf.xacro (robot description, xacro)
@@ -47,6 +47,6 @@
           filename="${meshes_file_directory}/Base.STL" />
       </geometry>
-      <material name="brightyellow" >
-        <color rgba="1.0 0.9921568627450981 0.00392156862745098 1.0" />
+      <material name="brightyellow">
+        <color rgba="1.0 1.0 1.0 1.0" />
       </material>
     </visual>
@@ -85,6 +85,6 @@
           filename="${meshes_file_directory}/Shoulder_Rotation_Pitch.STL" />
       </geometry>
-      <material name="brightyellow" >
-        <color rgba="1.0 0.9921568627450981 0.00392156862745098 1.0" />
+      <material name="brightyellow">
+        <color rgba="1.0 1.0 1.0 1.0" />
       </material>
     </visual>
@@ -136,6 +136,6 @@
           filename="${meshes_file_directory}/Upper_Arm.STL" />
       </geometry>
-      <material name="brightyellow" >
-        <color rgba="1.0 0.9921568627450981 0.00392156862745098 1.0" />
+      <material name="brightyellow">
+        <color rgba="1.0 1.0 1.0 1.0" />
       </material>
     </visual>
@@ -187,6 +187,6 @@
           filename="${meshes_file_directory}/Lower_Arm.STL" />
       </geometry>
-      <material name="brightyellow" >
-        <color rgba="1.0 0.9921568627450981 0.00392156862745098 1.0" />
+      <material name="brightyellow">
+        <color rgba="1.0 1.0 1.0 1.0" />
       </material>
     </visual>
@@ -238,6 +238,6 @@
           filename="${meshes_file_directory}/Wrist_Pitch_Roll.STL" />
       </geometry>
-      <material name="brightyellow" >
-        <color rgba="1.0 0.9921568627450981 0.00392156862745098 1.0" />
+      <material name="brightyellow">
+        <color rgba="1.0 1.0 1.0 1.0" />
       </material>
     </visual>
@@ -289,6 +289,6 @@
           filename="${meshes_file_directory}/Fixed_Gripper.STL" />
       </geometry>
-      <material name="brightyellow" >
-        <color rgba="1.0 0.9921568627450981 0.00392156862745098 1.0" />
+      <material name="brightyellow">
+        <color rgba="1.0 1.0 1.0 1.0" />
       </material>
     </visual>
@@ -340,6 +340,6 @@
           filename="${meshes_file_directory}/Moving_Jaw.STL" />
       </geometry>
-      <material name="brightyellow" >
-        <color rgba="1.0 0.9921568627450981 0.00392156862745098 1.0" />
+      <material name="brightyellow">
+        <color rgba="1.0 1.0 1.0 1.0" />
       </material>
     </visual>
@@ -374,6 +374,6 @@
         <box size="0.01 0.01 0.01" />
       </geometry>
-      <material name="red">
-        <color rgba="1.0 0.0 0.0 1"/>
+      <material name="brightyellow">
+        <color rgba="1.0 1.0 1.0 1.0" />
       </material>
     </visual>
