Commit message: arm moved

File: so_arm_100_description/urdf/so_arm_100_5dof.urdf.xacro (robot description, xacro)
@@ -3,7 +3,7 @@
   <xacro:arg name="prefix" default="" />
   <xacro:arg name="initial_positions_file" default="" />
-  <xacro:arg name="use_sim" default="false" />
+  <xacro:arg name="use_sim" default="true" />
   <xacro:arg name="use_topic_hardware_interface" default="false" />
-  <xacro:arg name="use_fake_hardware" default="true" />
+  <xacro:arg name="use_fake_hardware" default="false" />
   <xacro:arg name="ros2_control_type" default="so_arm_100_5dof_position" />
   <xacro:arg name="ros2_controllers_file" default="" />
@@ -11,20 +11,20 @@
   <xacro:include filename="$(find so_arm_100_description)/urdf/so_arm_100_5dof_arm.urdf.xacro" />
   <xacro:so_arm_100_5dof prefix="$(arg prefix)" />
-  <!-- Gazebo simulation -->
-  <xacro:if value="$(arg use_sim)">
-      <xacro:include filename="$(find so_arm_100_description)/urdf/so_arm_100_5dof.gazebo.xacro" />
-      <!-- fix the robot to the world -->
-      <link name="world"/>
-      <joint name="$(arg prefix)world_fixed" type="fixed">
-        <origin xyz="0 0 0" rpy="0 0 0"/>
-        <parent link="world"/>
-        <child link="$(arg prefix)base_link"/>
-      </joint>
-      <xacro:so_arm_100_5dof_gazebo
-        prefix="$(arg prefix)"
-        initial_positions_file="$(arg initial_positions_file)"
-        ros2_controllers_file="$(arg ros2_controllers_file)"
-        use_topic_hardware_interface="$(arg use_topic_hardware_interface)" />
-  </xacro:if>
+<!-- Gazebo simulation -->
+<!-- <xacro:if value="$(arg use_sim)"> -->
+    <!-- <xacro:include filename="$(find so_arm_100_description)/urdf/so_arm_100_5dof.gazebo.xacro" /> -->
+    <!-- fix the robot to the world -->
+    <!-- <link name="world"/> -->
+    <!-- <joint name="$(arg prefix)world_fixed" type="fixed"> -->
+      <!-- <origin xyz="0 0 0" rpy="0 0 0"/> -->
+      <!-- <parent link="world"/> -->
+      <!-- <child link="$(arg prefix)base_link"/> -->
+    <!-- </joint> -->
+    <!-- <xacro:so_arm_100_5dof_gazebo -->
+      <!-- prefix="$(arg prefix)" -->
+      <!-- initial_positions_file="$(arg initial_positions_file)" -->
+      <!-- ros2_controllers_file="$(arg ros2_controllers_file)" -->
+      <!-- use_topic_hardware_interface="$(arg use_topic_hardware_interface)" /> -->
+<!-- </xacro:if> -->
   <!-- ros2_control -->
   <xacro:include filename="$(find so_arm_100_description)/urdf/$(arg ros2_control_type).ros2_control.xacro" />

File: so_arm_100_description/urdf/so_arm_100_5dof_position.ros2_control.xacro (robot description, xacro)
@@ -38,5 +38,7 @@
           </xacro:if>
           <xacro:unless value="${use_topic_hardware_interface}">
-            <plugin>gz_ros2_control/GazeboSimSystem</plugin>
+            <!-- <plugin>gz_ros2_control/GazeboSimSystem</plugin> -->
+            <plugin>mujoco_ros2_control/MujocoSystemInterface</plugin>
+            <param name="mujoco_model">/home/deviant/so101_moveit_ws/src/so101_mujoco/scene.xml</param>
           </xacro:unless>
         </xacro:if>

File: so_arm_100_moveit_config/config/so_arm_100.ros2_control.xacro (robot description, xacro)
@@ -6,5 +6,7 @@
             <hardware>
                 <xacro:if value="${use_fake_hardware}">
-                    <plugin>mock_components/GenericSystem</plugin>
+                    <!-- <plugin>mock_components/GenericSystem</plugin> -->
+                    <plugin>mujoco_ros2_control/MujocoSystemInterface</plugin>
+                    <param name="mujoco_model">/home/deviant/so101_moveit_ws/src/so101_mujoco/scene.xml</param>
                 </xacro:if>
                 <xacro:unless value="${use_fake_hardware}">
