Commit message: path fixes

File: so_arm_100_description/urdf/so_arm_100_5dof.urdf.xacro (robot description, xacro)
@@ -8,4 +8,5 @@
   <xacro:arg name="ros2_control_type" default="so_arm_100_5dof_position" />
   <xacro:arg name="ros2_controllers_file" default="" />
+  <xacro:arg name="mujoco_model" default="" />
   <!-- so_arm_100 -->
   <xacro:include filename="$(find so_arm_100_description)/urdf/so_arm_100_5dof_arm.urdf.xacro" />
@@ -34,4 +35,5 @@
     use_sim="$(arg use_sim)"
     use_topic_hardware_interface="$(arg use_topic_hardware_interface)"
-    use_fake_hardware="$(arg use_fake_hardware)" />
+    use_fake_hardware="$(arg use_fake_hardware)"
+    mujoco_model="$(arg mujoco_model)" />
 </robot>

File: so_arm_100_description/urdf/so_arm_100_5dof_position.ros2_control.xacro (robot description, xacro)
@@ -9,4 +9,5 @@
       use_topic_hardware_interface:=^|false
       use_fake_hardware:=^|false
+      mujoco_model:=^|''
       serial_port:=^|/dev/ttyUSB0
       serial_baudrate:=^|1000000
@@ -40,5 +41,5 @@
             <!-- <plugin>gz_ros2_control/GazeboSimSystem</plugin> -->
             <plugin>mujoco_ros2_control/MujocoSystemInterface</plugin>
-            <param name="mujoco_model">/home/deviant/so101_moveit_ws/src/so101_mujoco/scene.xml</param>
+            <param name="mujoco_model">${mujoco_model}</param>
           </xacro:unless>
         </xacro:if>

File: so_arm_100_moveit_config/config/so_arm_100.ros2_control.xacro (robot description, xacro)
@@ -1,5 +1,5 @@
 <?xml version="1.0"?>
 <robot xmlns:xacro="http://www.ros.org/wiki/xacro">
-    <xacro:macro name="so_arm_100_ros2_control" params="name initial_positions_file use_fake_hardware serial_port:=^|/dev/ttyUSB0 serial_baudrate:=^|1000000 servo_speed:=^|2400 servo_acceleration:=^|50" >
+    <xacro:macro name="so_arm_100_ros2_control" params="name initial_positions_file use_fake_hardware mujoco_model:=^|'' serial_port:=^|/dev/ttyUSB0 serial_baudrate:=^|1000000 servo_speed:=^|2400 servo_acceleration:=^|50" >
         <xacro:property name="initial_positions" value="${xacro.load_yaml(initial_positions_file)['initial_positions']}"/>
         <ros2_control name="${name}" type="system">
@@ -8,5 +8,5 @@
                     <!-- <plugin>mock_components/GenericSystem</plugin> -->
                     <plugin>mujoco_ros2_control/MujocoSystemInterface</plugin>
-                    <param name="mujoco_model">/home/deviant/so101_moveit_ws/src/so101_mujoco/scene.xml</param>
+                    <param name="mujoco_model">${mujoco_model}</param>
                 </xacro:if>
                 <xacro:unless value="${use_fake_hardware}">

File: so_arm_100_moveit_config/config/so_arm_100.urdf.xacro (robot description, xacro)
@@ -4,4 +4,5 @@
     <xacro:arg name="initial_positions_file" default="initial_positions.yaml" />
     <xacro:arg name="use_fake_hardware" default="false"/>
+    <xacro:arg name="mujoco_model" default=""/>
     <xacro:arg name="serial_port" default="/dev/ttyUSB0"/>
     <xacro:arg name="serial_baudrate" default="1000000"/>
@@ -17,4 +18,5 @@
         initial_positions_file="$(arg initial_positions_file)"
         use_fake_hardware="$(arg use_fake_hardware)"
+        mujoco_model="$(arg mujoco_model)"
         serial_port="$(arg serial_port)"
         serial_baudrate="$(arg serial_baudrate)"
