Commit message: moveit new pacakge

File: so_arm_100_moveit_config/config/so_arm_100.ros2_control.xacro (robot description, xacro)
@@ -1,52 +1,79 @@
 <?xml version="1.0"?>
 <robot xmlns:xacro="http://www.ros.org/wiki/xacro">
-    <xacro:macro name="so_arm_100_5dof_ros2_control" params="name initial_positions_file">
-        <xacro:property name="initial_positions" value="${load_yaml(initial_positions_file)['initial_positions']}"/>
+    <xacro:macro name="so_arm_100_ros2_control" params="name initial_positions_file use_fake_hardware serial_port:=^|/dev/ttyUSB0 serial_baudrate:=^|1000000 servo_speed:=^|2400 servo_acceleration:=^|50" >
+        <xacro:property name="initial_positions" value="${xacro.load_yaml(initial_positions_file)['initial_positions']}"/>
         <ros2_control name="${name}" type="system">
             <hardware>
-                <!-- By default, set up controllers for simulation. This won't work on real hardware -->
-                <plugin>mock_components/GenericSystem</plugin>
+                <xacro:if value="${use_fake_hardware}">
+                    <plugin>mock_components/GenericSystem</plugin>
+                </xacro:if>
+                <xacro:unless value="${use_fake_hardware}">
+                    <plugin>so_arm_100_controller/SOARM100Interface</plugin>
+                    <param name="use_serial">true</param>
+                    <param name="serial_port">${serial_port}</param>
+                    <param name="serial_baudrate">${serial_baudrate}</param>
+                    <param name="servo_speed">${servo_speed}</param>
+                    <param name="servo_acceleration">${servo_acceleration}</param>
+                </xacro:unless>
             </hardware>
             <joint name="Shoulder_Rotation">
                 <command_interface name="position"/>
+                <command_interface name="velocity"/>
+                <command_interface name="effort"/>
                 <state_interface name="position">
                   <param name="initial_value">${initial_positions['Shoulder_Rotation']}</param>
                 </state_interface>
                 <state_interface name="velocity"/>
+                <state_interface name="effort"/>
             </joint>
             <joint name="Shoulder_Pitch">
                 <command_interface name="position"/>
+                <command_interface name="velocity"/>
+                <command_interface name="effort"/>
                 <state_interface name="position">
                   <param name="initial_value">${initial_positions['Shoulder_Pitch']}</param>
                 </state_interface>
                 <state_interface name="velocity"/>
+                <state_interface name="effort"/>
             </joint>
             <joint name="Elbow">
                 <command_interface name="position"/>
+                <command_interface name="velocity"/>
+                <command_interface name="effort"/>
                 <state_interface name="position">
                   <param name="initial_value">${initial_positions['Elbow']}</param>
                 </state_interface>
                 <state_interface name="velocity"/>
+                <state_interface name="effort"/>
             </joint>
             <joint name="Wrist_Pitch">
                 <command_interface name="position"/>
+                <command_interface name="velocity"/>
+                <command_interface name="effort"/>
                 <state_interface name="position">
                   <param name="initial_value">${initial_positions['Wrist_Pitch']}</param>
                 </state_interface>
                 <state_interface name="velocity"/>
+                <state_interface name="effort"/>
             </joint>
             <joint name="Wrist_Roll">
                 <command_interface name="position"/>
+                <command_interface name="velocity"/>
+                <command_interface name="effort"/>
                 <state_interface name="position">
                   <param name="initial_value">${initial_positions['Wrist_Roll']}</param>
                 </state_interface>
                 <state_interface name="velocity"/>
+                <state_interface name="effort"/>
             </joint>
             <joint name="Gripper">
                 <command_interface name="position"/>
+                <command_interface name="velocity"/>
+                <command_interface name="effort"/>
                 <state_interface name="position">
                   <param name="initial_value">${initial_positions['Gripper']}</param>
                 </state_interface>
                 <state_interface name="velocity"/>
+                <state_interface name="effort"/>
             </joint>
         </ros2_control>
